Commit message: fillin the contain of urdf, assembly not include

File: src/lily_description/urdf/mech/base.urdf.xacro (robot description, xacro)
@@ -1,5 +1,51 @@
 <?xml version="1.0"?>
 <robot xmlns:xacro="http://ros.org/wiki/xacro">
-<xacro:macro name="base" params="length width height mass">
-</xacro:macro>
+    <xacro:macro name="base" params="length width height mass wheel_radius wheel_pos_z">
+        <link name="base_footprint" />
+        <link name="base_link">
+            <visual>
+                <origin xyz="0 0 0" rpy="0 0 0" />
+                <geometry>
+                    <xacro:if value="${mesh_file == ''}">
+                        <box size="${length} ${width} ${height}" />
+                    </xacro:if>
+                    <xacro:unless value="${mesh_file == ''}">
+                        <mesh filename="${mesh_file}" scale="1 1 1" />
+                    </xacro:unless>
+                </geometry>
+                <material name="yellow">
+                    <color rgba="0.8784 0.6627 0.6627 1.0" />
+                </material>
+            </visual>
+            <collision>
+                <origin xyz="0 0 0" rpy="0 0 0" />
+                <geometry>
+                    <box size="${length} ${width} ${height}" />
+                </geometry>
+            </collision>
+            <inertial>
+                <origin xyz="0 0 0" rpy="0 0 0" />
+                <mass value="${mass}" />
+                <inertia ixx="${(1/12) * mass * ((width  * width)  + (height * height))}" ixy="0.0"
+                    ixz="0.0"
+                    iyy="${(1/12) * mass * ((length * length) + (height * height))}" iyz="0.0"
+                    izz="${(1/12) * mass * ((length * length) + (width  * width))}" />
+            </inertial>
+        </link>
+        <gazebo reference="base_link">
+            <visual>
+                <material>
+                    <ambient>0.8392 0.6314 0.0 1.0</ambient>
+                    <diffuse>0.8392 0.6314 0.0 1.0</diffuse>
+                    <specular>0.99 0.99 0.99 1.0</specular>
+                    <emissive>0.0 0.0 0.0 0.0</emissive>
+                </material>
+            </visual>
+        </gazebo>
+        <joint name="base_to_footprint" type="fixed">
+            <parent link="base_footprint" />
+            <child link="base_link" />
+            <origin xyz="0 0 0" rpy="0 0 0" />
+        </joint>
+    </xacro:macro>
 </robot>

File: src/lily_description/urdf/mech/joint.urdf.xacro (robot description, xacro)
@@ -1,3 +1,44 @@
 <?xml version="1.0"?>
 <robot xmlns:xacro="http://ros.org/wiki/xacro">
+    <xacro:macro name="joint" params="frame_id parent pos_x pos_y pos_z">
+        <link name="{side}_joint_link">
+            <visual>
+                <origin xyz="0 0 0" rpy="${pi/2} 0 0" />
+                <geometry>
+                    <box size="${length} ${width} ${height}" />
+                </geometry>
+                <material name="yellow">
+                    <color rgba="0.0 0.0 0.6627 1.0" />
+                </material>
+            </visual>
+            <collision>
+                <origin xyz="0 0 0" rpy="0 0 0" />
+                <geometry>
+                    <box size="${length} ${width} ${height}" />
+                </geometry>
+            </collision>
+            <inertial>
+                <origin xyz="0 0 0" rpy="0 0 0" />
+                <mass value="${mass}" />
+                <inertia ixx="${(1/12) * mass * ((width  * width)  + (height * height))}" ixy="0.0"
+                    ixz="0.0"
+                    iyy="${(1/12) * mass * ((length * length) + (height * height))}" iyz="0.0"
+                    izz="${(1/12) * mass * ((length * length) + (width  * width))}" />
+            </inertial>
+        </link>
+        <gazebo reference="base_link">
+            <visual>
+                <material>
+                    <ambient>0.8392 0.6314 0.0 1.0</ambient>
+                    <diffuse>0.8392 0.6314 0.0 1.0</diffuse>
+                    <specular>0.99 0.99 0.99 1.0</specular>
+                    <emissive>0.0 0.0 0.0 0.0</emissive>
+                </material>base_to_footprint </visual>
+        </gazebo>
+        <joint name="${frame_id}_joint" type="revolute">
+            <parent link="${parent}" />
+            <child link="${frame_id}_joint_link" />
+            <origin xyz="0 0 0" rpy="0 0 0" />
+        </joint>
+    </xacro:macro>
 </robot>

File: src/lily_description/urdf/mech/wheel.urdf.xacro (robot description, xacro)
@@ -1,3 +1,50 @@
 <?xml version="1.0"?>
 <robot xmlns:xacro="http://ros.org/wiki/xacro">
+    <xacro:macro name="wheel" params="side radius width pos_x pos_y pos_z mass">
+        <link name="{side}_wheel_link">
+            <visual>
+                <origin xyz="0 0 0" rpy="${pi/2} 0 0" />
+                <geometry>
+                    <xacro:if value="${mesh_file == ''}">
+                        <cylinder radius="${radius}" length="${width}" />
+                    </xacro:if>
+                    <xacro:unless value="${mesh_file == ''}">
+                        <mesh filename="${mesh_file}" scale="1 1 1" />
+                    </xacro:unless>
+                </geometry>
+                <material name="blue">
+                    <color rgba="0.1764 0.4588 0.8509 1.0" />
+                </material>
+            </visual>
+            <collision>
+                <origin xyz="0 0 0" rpy="${pi/2} 0 0" />
+                <geometry>
+                    <cylinder radius="${radius}" length="${width}" />
+                </geometry>
+            </collision>
+            <inertial>
+                <origin xyz="0 0 0" rpy="0 0 0" />
+                <mass value="${mass}" />
+                <inertia ixx="${(2/5) * mass * (radius * radius)}" ixy="0" ixz="0"
+                    iyy="${(2/5) * mass * (radius * radius)}" iyz="0"
+                    izz="${(2/5) * mass * (radius * radius)}" />
+            </inertial>
+        </link>
+        <gazebo reference="${side}_wheel_link">
+            <visual>
+                <material>
+                    <ambient>0.1764 0.4588 0.8509 1.0</ambient>
+                    <diffuse>0.1764 0.4588 0.8509 1.0</diffuse>
+                    <specular>0.1764 0.4588 0.8509 1.0</specular>
+                    <emissive>0.0 0.0 0.0 0.0</emissive>
+                </material>
+            </visual>
+        </gazebo>
+        <joint name="${side}_wheel_joint" type="continuous">
+            <axis xyz="0 1 0" />
+            <parent link="base_link" />
+            <child link="${side}_wheel_link" />
+            <origin xyz="${pos_x} ${pos_y} ${pos_z}" rpy="0 0 0" />
+        </joint>
+    </xacro:macro>
 </robot>

File: src/lily_description/urdf/robot.urdf.xacro (robot description, xacro)
@@ -1,3 +1,35 @@
 <?xml version="1.0"?>
 <robot xmlns:xacro="http://ros.org/wiki/xacro">
+    <!-- INCLUDE -->
+    <xacro:include filename="$(find lily_description)/urdf/mech/base.urdf.xacro" />
+    <xacro:include filename="$(find lily_description)/urdf/mech/wheel.urdf.xacro" />
+    <xacro:include filename="$(find lily_description)/urdf/sensors/plugins.urdf.xacro" />
+    <xacro:include filename="$(find lily_description)/urdf/sensors/imu.urdf.xacro" />
+    <xacro:include filename="$(find lily_description)/urdf/sensors/lidar.urdf.xacro" />
+    <xacro:include filename="$(find lily_description)/urdf/sensors/camera.urdf.xacro" />
+    <!-- DECLARATION -->
+    <xacro:property name="base_length" value="0.445" />
+    <xacro:property name="base_width" value="0.200" />
+    <xacro:property name="base_height" value="0.129" />
+    <xacro:property name="base_mass" value="10" />
+    <xacro:property name="wheel_radius" value="0.07162" />
+    <xacro:property name="wheel_width" value="0.05" />
+    <xacro:property name="wheel_pos_x" value="0.120" />
+    <xacro:property name="wheel_pos_y" value="0.1355" />
+    <xacro:property name="wheel_pos_z" value="-0.04788" />
+    <xacro:property name="wheel_mass" value=".6" />
+    <xacro:property name="wheel_torque" value="20" />
+    <!-- FUNCTION(SETUP) -->
+    <xacro:base
+        length="${base_length}"
+        width="${base_width}"
+        height="${base_height}"
+        mass="${base_mass}"
+        wheel_radius="${wheel_radius}"
+        wheel_pos_z="${wheel_pos_z}"
+    />
+    <xacro:depth_sensor name="eye">
+        <origin xyz="-0.065 0 0.255" rpy="0 0 0" />
+    </xacro:depth_sensor>
+    <xacro:imu />
 </robot>

Commit message: able to run the model, but fail at assembly

File: src/lily_description/urdf/mech/base.urdf.xacro (robot description, xacro)
@@ -7,10 +7,5 @@
                 <origin xyz="0 0 0" rpy="0 0 0" />
                 <geometry>
-                    <xacro:if value="${mesh_file == ''}">
-                        <box size="${length} ${width} ${height}" />
-                    </xacro:if>
-                    <xacro:unless value="${mesh_file == ''}">
-                        <mesh filename="${mesh_file}" scale="1 1 1" />
-                    </xacro:unless>
+                    <box size="${length} ${width} ${height}" />
                 </geometry>
                 <material name="yellow">

File: src/lily_description/urdf/mech/joint.urdf.xacro (robot description, xacro)
@@ -2,5 +2,9 @@
 <robot xmlns:xacro="http://ros.org/wiki/xacro">
     <xacro:macro name="joint" params="frame_id parent pos_x pos_y pos_z">
-        <link name="{side}_joint_link">
+        <xacro:property name="length" value="10" />
+        <xacro:property name="width" value="3" />
+        <xacro:property name="height" value="3" />
+        <xacro:property name="mass" value="3" />
+        <link name="${frame_id}_joint_link">
             <visual>
                 <origin xyz="0 0 0" rpy="${pi/2} 0 0" />
@@ -40,4 +44,8 @@
             <child link="${frame_id}_joint_link" />
             <origin xyz="0 0 0" rpy="0 0 0" />
+            <limit lower="-1.57"
+                upper="1.57"
+                effort="50"
+                velocity="5.0" />
         </joint>
     </xacro:macro>

File: src/lily_description/urdf/mech/wheel.urdf.xacro (robot description, xacro)
@@ -6,10 +6,5 @@
                 <origin xyz="0 0 0" rpy="${pi/2} 0 0" />
                 <geometry>
-                    <xacro:if value="${mesh_file == ''}">
-                        <cylinder radius="${radius}" length="${width}" />
-                    </xacro:if>
-                    <xacro:unless value="${mesh_file == ''}">
-                        <mesh filename="${mesh_file}" scale="1 1 1" />
-                    </xacro:unless>
+                    <cylinder radius="${radius}" length="${width}" />
                 </geometry>
                 <material name="blue">

File: src/lily_description/urdf/robot.urdf.xacro (robot description, xacro)
@@ -1,5 +1,6 @@
 <?xml version="1.0"?>
-<robot xmlns:xacro="http://ros.org/wiki/xacro">
+<robot name="lily" xmlns:xacro="http://ros.org/wiki/xacro">
     <!-- INCLUDE -->
+    <xacro:include filename="$(find lily_description)/urdf/mech/joint.urdf.xacro" />
     <xacro:include filename="$(find lily_description)/urdf/mech/base.urdf.xacro" />
     <xacro:include filename="$(find lily_description)/urdf/mech/wheel.urdf.xacro" />
@@ -9,6 +10,6 @@
     <xacro:include filename="$(find lily_description)/urdf/sensors/camera.urdf.xacro" />
     <!-- DECLARATION -->
-    <xacro:property name="base_length" value="0.445" />
-    <xacro:property name="base_width" value="0.200" />
+    <xacro:property name="base_length" value="0.200" />
+    <xacro:property name="base_width" value="0.445" />
     <xacro:property name="base_height" value="0.129" />
     <xacro:property name="base_mass" value="10" />
@@ -20,4 +21,7 @@
     <xacro:property name="wheel_mass" value=".6" />
     <xacro:property name="wheel_torque" value="20" />
+    <xacro:property name="thigh_pos_x" value="${base_width/2}" />
+    <xacro:property name="thigh_pos_y" value="0" />
+    <xacro:property name="thigh_pos_z" value="0" />
     <!-- FUNCTION(SETUP) -->
     <xacro:base
@@ -29,6 +33,12 @@
         wheel_pos_z="${wheel_pos_z}"
     />
+    <xacro:joint
+        frame_id="left_thigh"
+        parent="base_link"
+        pos_x="${thigh_pos_x}"
+        pos_y="${thigh_pos_y}"
+        pos_z="${thigh_pos_z}" />
     <xacro:depth_sensor name="eye">
-        <origin xyz="-0.065 0 0.255" rpy="0 0 0" />
+        <origin xyz="${base_length/2} 0 ${base_height/2}" rpy="0 0 0" />
     </xacro:depth_sensor>
     <xacro:imu />
