Commit message: update 3d wheel

File: src/lily_description/urdf/mechanic_part/wheel.urdf.xacro (robot description, xacro)
@@ -6,9 +6,10 @@
                 <origin xyz="0 0 0" rpy="${pi/2} 0 0" />
                 <geometry>
-                    <cylinder radius="${radius}" length="${width}" />
+                    <!-- <cylinder radius="${radius}" length="${width}" /> -->
+                    <mesh filename="file://$(find lily_description)/meshes/tire.dae" scale="4 4 4" />
                 </geometry>
-                <material name="blue">
+                <!-- <material name="blue">
                     <color rgba="0.1764 0.4588 0.8509 1.0" />
-                </material>
+                </material> -->
             </visual>
             <collision>
