Commit message: able to move the joint

File: src/lily_description/urdf/mechanic_part/base.urdf.xacro (robot description, xacro)
@@ -1,5 +1,5 @@
 <?xml version="1.0"?>
 <robot xmlns:xacro="http://ros.org/wiki/xacro">
-    <xacro:macro name="base" params="length width height mass wheel_radius wheel_pos_z">
+    <xacro:macro name="base" params="length width height mass">
         <link name="base_footprint" />
         <link name="base_link">

File: src/lily_description/urdf/mechanic_part/knee.urdf.xacro (robot description, xacro)
@@ -42,5 +42,5 @@
             <origin xyz="${pos_x - (length/2)} ${pos_y} ${pos_z}" rpy="0 0 0" />
             <axis xyz="0 1 0" />
-            <limit lower="-1.57"
+            <limit lower="-3.14"
                 upper="1.57"
                 effort="50"

File: src/lily_description/urdf/robot.urdf.xacro (robot description, xacro)
@@ -10,4 +10,5 @@
     <xacro:include filename="$(find lily_description)/urdf/sensors/lidar.urdf.xacro" />
     <xacro:include filename="$(find lily_description)/urdf/sensors/camera.urdf.xacro" />
+    <xacro:include filename="$(find lily_description)/urdf/controller/ros2_control.urdf.xacro" />
     <!-- DECLARATION -->
     <xacro:property name="base_length" value="0.200" />
@@ -17,7 +18,4 @@
     <xacro:property name="wheel_radius" value="0.09" />
     <xacro:property name="wheel_width" value="0.05" />
-    <xacro:property name="wheel_pos_x" value="0.120" />
-    <xacro:property name="wheel_pos_y" value="0.1355" />
-    <xacro:property name="wheel_pos_z" value="-0.04788" />
     <xacro:property name="wheel_mass" value=".6" />
     <xacro:property name="wheel_torque" value="20" />
@@ -26,7 +24,8 @@
     <xacro:property name="thigh_height" value="0.07" />
     <xacro:property name="thigh_pos_x" value="${thigh_length/2}" />
-    <xacro:property name="thigh_pos_y" value="${base_width/2}" />
+    <xacro:property name="thigh_pos_y" value="${(base_width/2) + (thigh_width/2)}" />
     <xacro:property name="thigh_pos_z" value="0" />
     <!-- FUNCTION(SETUP) -->
+    <xacro:lily_ros2_control />
     <xacro:base
         length="${base_length}"
@@ -34,6 +33,4 @@
         height="${base_height}"
         mass="${base_mass}"
-        wheel_radius="${wheel_radius}"
-        wheel_pos_z="${wheel_pos_z}"
     />
     <xacro:thigh
@@ -60,6 +57,6 @@
         frame_id="left_knee"
         parent="left_thigh"
-        pos_x="${thigh_length+(thigh_length/2)}"
-        pos_y="0"
+        pos_x="${(thigh_length+(thigh_length/2))-thigh_width}"
+        pos_y="${thigh_width/2}"
         pos_z="0"
         length="${thigh_length}"
@@ -70,6 +67,6 @@
         frame_id="right_knee"
         parent="right_thigh"
-        pos_x="${thigh_length+(thigh_length/2)}"
-        pos_y="0"
+        pos_x="${(thigh_length+(thigh_length/2))-thigh_width}"
+        pos_y="${-thigh_width/2}"
         pos_z="0"
         length="${thigh_length}"
