Commit message: update: adding bt, controlling the robot like servo, combining servo joint so it can be use in while loop

File: src/lily_description/urdf/mechanic_part/knee.urdf.xacro (robot description, xacro)
@@ -44,5 +44,5 @@
             <limit lower="-3.14"
                 upper="1.57"
-                effort="50"
+                effort="100"
                 velocity="5.0" />
         </joint>

File: src/lily_description/urdf/mechanic_part/thigh.urdf.xacro (robot description, xacro)
@@ -44,5 +44,5 @@
             <limit lower="0.0"
                 upper="3.14"
-                effort="50"
+                effort="100"
                 velocity="5.0" />
         </joint>

File: src/lily_description/urdf/mechanic_part/wheel.urdf.xacro (robot description, xacro)
@@ -28,10 +28,5 @@
         <gazebo reference="${side}_wheel_link">
             <visual>
-                <material>
-                    <ambient>0.1764 0.4588 0.8509 1.0</ambient>
-                    <diffuse>0.1764 0.4588 0.8509 1.0</diffuse>
-                    <specular>0.1764 0.4588 0.8509 1.0</specular>
-                    <emissive>0.0 0.0 0.0 0.0</emissive>
-                </material>
+                <material>gazebo/Gray</material>
             </visual>
         </gazebo>

File: src/lily_description/urdf/robot.urdf.xacro (robot description, xacro)
@@ -85,4 +85,17 @@
         <origin xyz="${base_length/2} 0 ${base_height/2}" rpy="0 0 0" />
     </xacro:depth_sensor>
+    <xacro:laser
+        name="lidar"
+        parent ="base_link"
+        update_rate="10"
+        ray_count="64"
+        min_angle="-1.39626340159"
+        max_angle="1.39626340159"
+        min_range="0.1"
+        max_range="10.0"
+        frame_id="lidar_link"
+        topic_name="/scan">
+        <origin xyz="0 0 ${(base_height/2) -  0.025 }" rpy="0 0 0" />
+    </xacro:laser>
     <xacro:imu />
 </robot>

File: src/lily_description/urdf/sensors/lidar.urdf.xacro (robot description, xacro)
@@ -3,8 +3,8 @@
     <xacro:property name="M_PI" value="3.1415926535897931" />
     <xacro:macro name="laser"
-        params="name pos_x pos_y pos_z update_rate ray_count min_angle max_angle min_range max_range frame_id topic_name">
-        <link name="$frame_id}">
+        params="name parent *origin update_rate ray_count min_angle max_angle min_range max_range frame_id topic_name">
+        <link name="${frame_id}">
             <visual>
-                <origin xyz="0 0 -0.025" rpy="0 0 0" />
+                <xacro:insert_block name="origin" />
                 <geometry>
                     <cylinder radius="0.0375" length="0.05" />
@@ -15,5 +15,5 @@
             </visual>
             <collision>
-                <origin xyz="0 0 -0.025" rpy="0 0 0" />
+                <xacro:insert_block name="origin" />
                 <geometry>
                     <cylinder radius="0.0375" length="0.05" />
@@ -39,5 +39,5 @@
         </gazebo>
         <joint name="${frame_id}_to_base_link" type="fixed">
-            <parent link="base_link" />
+            <parent link="${parent}" />
             <child link="${frame_id}" />
             <xacro:insert_block name="origin" />
@@ -61,6 +61,6 @@
                             <samples>1</samples>
                             <resolution>1</resolution>
-                            <min_angle>0.0</min_angle>
-                            <max_angle>0.0</max_angle>
+                            <min_angle>-0.2618</min_angle>
+                            <max_angle>0.2618</max_angle>
                         </vertical>
                     </scan>
