Commit message: change of name

File: src/arc_description/urdf/controller/diff_drive.urdf.xacro (robot description, xacro)
@@ -1,7 +1,7 @@
 <?xml version="1.0"?>
 <robot xmlns:xacro="http://ros.org/wiki/xacro">
-    <xacro:include filename="$(find lily_description)/urdf/declaration.urdf.xacro" />
-    <xacro:macro name="lily_diff_drive_control">
-        <ros2_control name="LilyDiffDriveSystem" type="system">
+    <xacro:include filename="$(find arc_description)/urdf/declaration.urdf.xacro" />
+    <xacro:macro name="arc_diff_drive_control">
+        <ros2_control name="arcDiffDriveSystem" type="system">
             <hardware>
                 <plugin>gz_ros2_control/GazeboSimSystem</plugin>  <!-- ← real Gazebo connection -->

File: src/arc_description/urdf/controller/ros2_control.urdf.xacro (robot description, xacro)
@@ -1,6 +1,6 @@
 <?xml version="1.0"?>
 <robot xmlns:xacro="http://ros.org/wiki/xacro">
-    <xacro:macro name="lily_ros2_control">
-        <ros2_control name="LilySystem" type="system">
+    <xacro:macro name="arc_ros2_control">
+        <ros2_control name="arcSystem" type="system">
             <hardware>
                 <plugin>gz_ros2_control/GazeboSimSystem</plugin>  <!-- ← real Gazebo connection -->
@@ -38,5 +38,5 @@
             <plugin filename="gz_ros2_control-system"
                 name="gz_ros2_control::GazeboSimROS2ControlPlugin">
-                <parameters>$(find lily_description)/config/controllers.yaml</parameters>
+                <parameters>$(find arc_description)/config/controllers.yaml</parameters>
             </plugin>
         </gazebo>

File: src/arc_description/urdf/declaration.urdf.xacro (robot description, xacro)
@@ -1,4 +1,4 @@
 <?xml version="1.0"?>
-<robot name="lily" xmlns:xacro="http://ros.org/wiki/xacro">
+<robot name="arc" xmlns:xacro="http://ros.org/wiki/xacro">
     <!-- DECLARATION -->
     <xacro:property name="base_length" value="0.200" />

File: src/arc_description/urdf/mechanic_part/wheel.urdf.xacro (robot description, xacro)
@@ -7,5 +7,5 @@
                 <geometry>
                     <!-- <cylinder radius="${radius}" length="${width}" /> -->
-                    <mesh filename="file://$(find lily_description)/meshes/tire.dae" scale="4 4 4" />
+                    <mesh filename="file://$(find arc_description)/meshes/tire.dae" scale="4 4 4" />
                 </geometry>
                 <!-- <material name="blue">

File: src/arc_description/urdf/robot.urdf.xacro (robot description, xacro)
@@ -1,19 +1,19 @@
 <?xml version="1.0"?>
-<robot name="lily" xmlns:xacro="http://ros.org/wiki/xacro">
+<robot name="arc" xmlns:xacro="http://ros.org/wiki/xacro">
     <!-- INCLUDE -->
-    <xacro:include filename="$(find lily_description)/urdf/declaration.urdf.xacro" />
-    <xacro:include filename="$(find lily_description)/urdf/mechanic_part/thigh.urdf.xacro" />
-    <xacro:include filename="$(find lily_description)/urdf/mechanic_part/knee.urdf.xacro" />
-    <xacro:include filename="$(find lily_description)/urdf/mechanic_part/base.urdf.xacro" />
-    <xacro:include filename="$(find lily_description)/urdf/mechanic_part/wheel.urdf.xacro" />
-    <xacro:include filename="$(find lily_description)/urdf/sensors/plugins.urdf.xacro" />
-    <xacro:include filename="$(find lily_description)/urdf/sensors/imu.urdf.xacro" />
-    <xacro:include filename="$(find lily_description)/urdf/sensors/lidar.urdf.xacro" />
-    <xacro:include filename="$(find lily_description)/urdf/sensors/camera.urdf.xacro" />
-    <xacro:include filename="$(find lily_description)/urdf/controller/ros2_control.urdf.xacro" />
-    <xacro:include filename="$(find lily_description)/urdf/controller/diff_drive.urdf.xacro" />
+    <xacro:include filename="$(find arc_description)/urdf/declaration.urdf.xacro" />
+    <xacro:include filename="$(find arc_description)/urdf/mechanic_part/thigh.urdf.xacro" />
+    <xacro:include filename="$(find arc_description)/urdf/mechanic_part/knee.urdf.xacro" />
+    <xacro:include filename="$(find arc_description)/urdf/mechanic_part/base.urdf.xacro" />
+    <xacro:include filename="$(find arc_description)/urdf/mechanic_part/wheel.urdf.xacro" />
+    <xacro:include filename="$(find arc_description)/urdf/sensors/plugins.urdf.xacro" />
+    <xacro:include filename="$(find arc_description)/urdf/sensors/imu.urdf.xacro" />
+    <xacro:include filename="$(find arc_description)/urdf/sensors/lidar.urdf.xacro" />
+    <xacro:include filename="$(find arc_description)/urdf/sensors/camera.urdf.xacro" />
+    <xacro:include filename="$(find arc_description)/urdf/controller/ros2_control.urdf.xacro" />
+    <xacro:include filename="$(find arc_description)/urdf/controller/diff_drive.urdf.xacro" />
     <!-- FUNCTION(SETUP) -->
-    <xacro:lily_ros2_control />
-    <xacro:lily_diff_drive_control />
+    <xacro:arc_ros2_control />
+    <xacro:arc_diff_drive_control />
     <xacro:base
         length="${base_length}"
